Commit message: feat: 使用 HI12 外置 IMU 替换 EP 内置 IMU
EP 内置 IMU 无磁力计、受电机干扰严重导致 yaw 漂移，
替换为 HiPNUC HI12 9轴 AHRS 提供绝对航向和更可靠的姿态数据。

- 新增 hi12_imu_node.py: HI12 串口驱动，解析 HiPNUC 二进制协议发布 /imu
- EP 驱动添加 enable_imu 参数，默认关闭 IMU 数据流和 /imu 发布
- EKF 配置 imu0_relative 改为 false（HI12 有磁力计绝对航向）
- URDF imu_link 位置更新为 HI12 安装位置
- launch 文件添加 HI12 节点启动和 use_hi12 参数切换
- .gitignore 添加 Temp/ 目录

Co-Authored-By: Claude Haiku 4.5 <noreply@anthropic.com>

File: src/rm_ep_description/urdf/rm_ep.urdf.xacro (robot description, xacro)
@@ -61,10 +61,12 @@
     </visual>
   </link>
-  <!-- ========== imu_link (底盘中心) ========== -->
+  <!-- ========== imu_link (HI12 外置 IMU，安装于底盘后方偏上) ========== -->
   <link name="imu_link"/>
   <joint name="imu_joint" type="fixed">
     <parent link="base_link"/>
     <child link="imu_link"/>
-    <origin xyz="0 0 ${chassis_height/2}" rpy="0 0 0"/>
+    <!-- HI12 安装位置: 底盘后方 (-0.08m)，居中 (0m)，底盘顶部偏上 (0.10m)
+         模块 X 轴朝前、Y 轴朝左、Z 轴朝上，与 base_link 对齐，rpy=0 -->
+    <origin xyz="-0.08 0 0.10" rpy="0 0 0"/>
   </joint>
   <!-- ========== laser_link (RPLIDAR A2 安装位置) ========== -->
