Commit message: fix: 修复 EKF 角速度融合、协方差、costmap 冲突、轮子参数四个 bug
- EKF: odom0_config vyaw 改为 false，HI12 模式下 odom angular.z=0 不再被融合
- EKF: initial_estimate_covariance 从 1e-9 改为合理值，避免锁死初始状态
- local_costmap: 删除 robot_radius 避免与 costmap_common 的 footprint 冲突
- URDF/驱动: wheel_radius=0.05, wheel_base=0.198, wheel_track=0.20 按实测值统一

File: src/rm_ep_description/urdf/rm_ep.urdf.xacro (robot description, xacro)
@@ -37,8 +37,8 @@
   <xacro:property name="chassis_height" value="0.10"/>
   <xacro:property name="chassis_clearance" value="0.045"/>
-  <xacro:property name="wheel_radius" value="0.0485"/>
+  <xacro:property name="wheel_radius" value="0.05"/>
   <xacro:property name="wheel_width" value="0.04"/>
-  <xacro:property name="wheel_base" value="0.24"/>
-  <xacro:property name="wheel_track" value="0.18"/>
+  <xacro:property name="wheel_base" value="0.198"/>
+  <xacro:property name="wheel_track" value="0.20"/>
   <!-- 激光雷达安装位置 (底盘顶部最前方居中) -->
   <xacro:property name="laser_x" value="0.11"/>

Commit message: feat(d435i): 添加 D435i 深度相机集成
- URDF 添加 d435i_link + d435i_joint
- 新建 realsense_d435i.launch 驱动封装
- 新建 d435i_depth_to_laser.launch 深度转激光扫描
- 新建 d435i_bringup.launch 独立启动（像键盘遥控一样）
- mapping/navigation 添加 use_d435i 参数支持内嵌启动
- 参数文件添加 D435i 配置
- package.xml 添加 ROS 依赖

File: src/rm_ep_description/urdf/rm_ep.urdf.xacro (robot description, xacro)
@@ -85,4 +85,15 @@
     <origin xyz="${laser_x} 0 ${chassis_height/2 + laser_z}" rpy="0 0 0"/>
   </joint>
+  <!-- ========== d435i_link (Intel RealSense D435i) ========== -->
+  <!-- 安装位置: 底盘顶部前方，激光雷达后方 -->
+  <xacro:property name="d435i_x" value="0.05"/>
+  <xacro:property name="d435i_y" value="0.0"/>
+  <xacro:property name="d435i_z" value="0.12"/>
+  <link name="d435i_link"/>
+  <joint name="d435i_joint" type="fixed">
+    <parent link="base_link"/>
+    <child link="d435i_link"/>
+    <origin xyz="${d435i_x} ${d435i_y} ${d435i_z}" rpy="0 0 0"/>
+  </joint>
   <!-- ========== 四个麦克纳姆轮 ========== -->
   <xacro:property name="pos_z" value="${-chassis_height/2 + wheel_radius + chassis_clearance}"/>

Commit message: fix(d435i): 修复 TF 挂载+同步文档+清理死参数
URDF: base_link→camera_link→d435i_link,让 realsense 发布的 camera_link 子树挂到机器人 TF 树(此前两棵树断开,/d435i/scan 坐标系错位)
文档: README/AGENTS/details/usage_guide TF 树更正为实际结构,README 补 D435i 用法,details 硬件表补 D435i 位置
params: 删除无 launch 引用的 d435i_* 死参数(realsense 2.3.2 裸 include)

File: src/rm_ep_description/urdf/rm_ep.urdf.xacro (robot description, xacro)
@@ -85,14 +85,24 @@
     <origin xyz="${laser_x} 0 ${chassis_height/2 + laser_z}" rpy="0 0 0"/>
   </joint>
-  <!-- ========== d435i_link (Intel RealSense D435i) ========== -->
+  <!-- ========== D435i (Intel RealSense D435i) ========== -->
   <!-- 安装位置: 底盘顶部前方，激光雷达后方 -->
   <xacro:property name="d435i_x" value="0.05"/>
   <xacro:property name="d435i_y" value="0.0"/>
   <xacro:property name="d435i_z" value="0.12"/>
+  <!-- camera_link: realsense2_camera 发布的 TF 子树根 (camera_link→camera_depth_frame→...)
+       驱动只发 camera_link 往下的子变换，不发 camera_link 的父变换，
+       所以这里由 URDF 把它挂到 base_link 上，二者接力、不冲突。 -->
+  <link name="camera_link"/>
+  <joint name="camera_link_joint" type="fixed">
+    <parent link="base_link"/>
+    <child link="camera_link"/>
+    <origin xyz="${d435i_x} ${d435i_y} ${d435i_z}" rpy="0 0 0"/>
+  </joint>
+  <!-- d435i_link: 语义别名, 挂在 camera_link 下, 给 depth_to_laserscan 的 output_frame_id 用 -->
   <link name="d435i_link"/>
-  <joint name="d435i_joint" type="fixed">
-    <parent link="base_link"/>
+  <joint name="d435i_link_joint" type="fixed">
+    <parent link="camera_link"/>
     <child link="d435i_link"/>
-    <origin xyz="${d435i_x} ${d435i_y} ${d435i_z}" rpy="0 0 0"/>
+    <origin xyz="0 0 0" rpy="0 0 0"/>
   </joint>
   <!-- ========== 四个麦克纳姆轮 ========== -->
